Commit message: Adding all the tasks

File: sahayak_bot/ebot_description/urdf/ebot.xacro (robot description, xacro)
@@ -13,5 +13,5 @@
     <inertial>
       <origin
-        xyz="0 -0.027412 0.07138"
+   xyz="0 0.0 0.12"
         rpy="0 0 0" />
       <mass
@@ -24,5 +24,5 @@
         iyz="-4.0532E-05"
         izz="0.030588" /> -->
-         <inertia ixx="6.68333333333" ixy="0" ixz="0" iyy="1.9722" iyz="0" izz="2.65266666667"/>
+         <inertia ixx="0.356" ixy="0" ixz="0" iyy="0.9443" iyz="0" izz="1.008"/>
     </inertial>
     <visual>
@@ -65,5 +65,5 @@
         iyz="3.3883E-09"
         izz="0.001221" /> -->
-          <inertia ixx="0.00285208333333" ixy="0" ixz="0" iyy="0.00285208333333" iyz="0" izz="0.005"/>
+          <inertia ixx="0.003" ixy="0" ixz="0" iyy="0.0030" iyz="0" izz="0.0035"/>
     </inertial>
     <visual>
@@ -119,5 +119,5 @@
         iyz="3.3744E-09"
         izz="0.001221" /> -->
-          <inertia ixx="0.00285208333333" ixy="0" ixz="0" iyy="0.00285208333333" iyz="0" izz="0.005"/>
+           <inertia ixx="0.003" ixy="0" ixz="0" iyy="0.0030" iyz="0" izz="0.0035"/>
     </inertial>
     <visual>
@@ -173,5 +173,5 @@
         iyz="3.3883E-09"
         izz="0.001221" /> -->
-          <inertia ixx="0.00285208333333" ixy="0" ixz="0" iyy="0.00285208333333" iyz="0" izz="0.005"/>
+           <inertia ixx="0.003" ixy="0" ixz="0" iyy="0.0030" iyz="0" izz="0.0035"/>
     </inertial>
     <visual>
@@ -227,5 +227,5 @@
         iyz="3.3744E-09"
         izz="0.001221" /> -->
-          <inertia ixx="0.00285208333333" ixy="0" ixz="0" iyy="0.00285208333333" iyz="0" izz="0.005"/>
+        <inertia ixx="0.003" ixy="0" ixz="0" iyy="0.0030" iyz="0" izz="0.0035"/>
     </inertial>
     <visual>
